Commit message: add endeffector offset for panda_pump

File: data/urdf/panda_pump.urdf (robot description, URDF)
Before this commit: robot panda_pump, 12 links, 11 joints
Links:
- added link panda_pump_ref
Joints:
- added joint panda_pump_joint_ref: type fixed, parent panda_pump, child panda_pump_ref, origin xyz=0 0 0.11 rpy=0 0 -0.7853981633974483

File: data/xacro/pump.xacro (robot description, xacro)
@@ -7,4 +7,9 @@
         <child link="${ns}_pump"/>
         <origin xyz="${xyz}" rpy="${rpy}"/>
+      </joint>
+      <joint name="${ns}_pump_joint_ref" type="fixed">
+        <parent link="${ns}_pump"/>
+        <child link="${ns}_pump_ref"/>
+        <origin rpy="0 0 -0.7853981633974483" xyz="0 0 0.11"/>
       </joint>
     </xacro:unless>
@@ -36,4 +41,25 @@
 <!--  scale="0.001 0.001 0.001" -->
     </link>
+    <link name="${ns}_pump_ref">
+        <!--collision>
+          <origin rpy="3.141592653589793 1.5707963267948966 1.5707963267948966" xyz="0.0424 0.0424 0.0"/>
+          <geometry>
+            <cylinder length="0.01" radius="0.06"/>
+          </geometry>
+        </collision>
+            <collision>
+      <origin rpy="0 0 0" xyz="0.0424 0.0424 -0.02"/>
+      <geometry>
+        <sphere radius="0.06"/>
+      </geometry>
+    </collision>
+    <collision>
+      <origin rpy="0 0 0" xyz="0.0424 0.0424 -0.03"/>
+      <geometry>
+        <sphere radius="0.06"/>
+      </geometry>
+    </collision-->
+    <!--  scale="0.001 0.001 0.001" -->
+    </link>
   </xacro:macro>
 </robot>
