Commit message: gripperstateadded

File: data/urdf/panda_hand.urdf (robot description, URDF)
Before this commit: robot panda_hand, 14 links, 13 joints
Links:
- added link panda_hand_ref
Joints:
- added joint panda_hnad_joint_ref: type fixed, parent panda_hand, child panda_hand_ref, origin xyz=0 0 0.10 rpy=0 0 0
- joint panda_hand_joint: origin xyz=0 0 0 rpy=0 0 -0.7853981633974483 -> xyz=0 0 0.1 rpy=0 0 -0.7853981633974483

File: data/xacro/hand.xacro (robot description, xacro)
@@ -8,4 +8,9 @@
         <child link="${ns}_hand"/>
         <origin xyz="${xyz}" rpy="${rpy}"/>
+      </joint>
+      <joint name="${ns}_hand_joint_ref" type="fixed">
+        <parent link="${ns}_hand"/>
+        <child link="${ns}_hand_ref"/>
+        <origin rpy="0 0 0.0" xyz="0 0 0.10"/>
       </joint>
     </xacro:unless>
@@ -90,4 +95,6 @@
       <mimic joint="${ns}_finger_joint1" />
     </joint>
+    <link name="${ns}_hand_ref">
+    </link>
   </xacro:macro>
 </robot>
