Commit message: add panda_fist for Impact manipulation experinces

File: data/urdf/panda_fist.urdf (robot description, URDF)
Before this commit: robot panda_pump, 13 links, 12 joints
Links:
- removed link panda_pump
- removed link panda_pump_ref
- added link panda_fist, mass 0.1; collision mesh filename=file://@URDF_DESTINATION@/meshes/fist.stl; visual mesh filename=file://@URDF_DESTINATION@/meshes/fist.stl
- added link panda_fist_ref
Joints:
- removed joint panda_pump_joint
- removed joint panda_pump_joint_ref
- added joint panda_fist_joint: type fixed, parent panda_link8, child panda_fist, origin xyz=0 0 0.055 rpy=0 0 -0.7853981633974483
- added joint panda_fist_ref: type fixed, parent panda_fist, child panda_fist_ref, origin xyz=0 0 0.055 rpy=0 0 0
