Commit message: panda_foot_ref

File: data/urdf/panda_foot.urdf (robot description, URDF)
Before this commit: robot panda_foot, 12 links, 11 joints
Links:
- added link panda_foot_ref
Joints:
- added joint panda_foot_joint_ref: type fixed, parent panda_foot, child panda_foot_ref, origin xyz=0 0 0.035 rpy=0 0 0

File: data/xacro/foot.xacro (robot description, xacro)
@@ -8,4 +8,14 @@
         <origin xyz="${xyz}" rpy="${rpy}"/>
       </joint>
+      <joint name="${ns}_foot_joint_ref" type="fixed">
+        <parent link="${ns}_foot"/>
+        <child link="${ns}_foot_ref"/>
+        <origin rpy="0 0 0.0" xyz="0 0 0.030"/>
+      </joint>
+      <!-- <joint name="${ns}_foot_joint_ref" type="fixed">
+        <parent link="${ns}_foot"/>
+        <child link="${ns}_foot_ref"/>
+        <origin rpy="0 0 0.0" xyz="0 0 0.035"/>
+      </joint> -->
     </xacro:unless>
     <xacro:arg name="gazebo" default="true"/>
@@ -35,4 +45,6 @@
       </collision>
     </link>
+    <link name="${ns}_foot_ref">
+    </link>
   </xacro:macro>
 </robot>
