Commit message: adding PushTool v1 + Foot modif

File: data/xacro/foot.xacro (robot description, xacro)
@@ -11,5 +11,5 @@
         <parent link="${ns}_foot"/>
         <child link="${ns}_foot_ref"/>
-        <origin rpy="0 0 0.0" xyz="0 0 0.030"/>
+        <origin rpy="0 0 0.0" xyz="0 0 0.02"/>
       </joint>
       <!-- <joint name="${ns}_foot_joint_ref" type="fixed">
