Commit message: Minor On PandaPush robot module- Adding New Poking Tool

File: data/xacro/panda_push.urdf.xacro (robot description, xacro)
@@ -9,4 +9,4 @@
   <xacro:main connected_to='world'/>
   <xacro:panda xyz="0 0 0" connected_to='main_link' safety_distance="0.03"/>
-  <xacro:push ns="panda" rpy="0 ${0} ${0}" xyz="0 0.00 0.008" connected_to="panda_link8"/>
+  <xacro:push ns="panda" rpy="0 ${0} ${0}" xyz="0 0.00 -0.000" connected_to="panda_link8"/>
 </robot>

File: data/xacro/push.xacro (robot description, xacro)
@@ -1,5 +1,5 @@
 <?xml version="1.0" encoding="utf-8"?>
 <robot xmlns:xacro="http://www.ros.org/wiki/xacro" name="panda_push_part">
-  <xacro:macro name="push" params="connected_to:='' ns:='' rpy:='0 0 0' xyz:='0.0 0.0 0.0' ">
+  <xacro:macro name="push" params="connected_to:='' ns:='' rpy:='0 0 0' xyz:='0.0 0.0 -0.1' ">
     <xacro:unless value="${connected_to == ''}">
       <joint name="${ns}_push_joint" type="fixed">
@@ -11,5 +11,5 @@
         <parent link="${ns}_push"/>
         <child link="${ns}_push_ref"/>
-        <origin rpy="0 0 0.0" xyz="0 0 0.143"/>
+        <origin rpy="0.0 0.0 0.0" xyz="0 0 0.2"/>
       </joint>
     </xacro:unless>

Commit message: minor panda_push

File: data/xacro/panda_push.urdf.xacro (robot description, xacro)
@@ -9,4 +9,4 @@
   <xacro:main connected_to='world'/>
   <xacro:panda xyz="0 0 0" connected_to='main_link' safety_distance="0.03"/>
-  <xacro:push ns="panda" rpy="0 ${0} ${0}" xyz="0 0.00 -0.000" connected_to="panda_link8"/>
+  <xacro:push ns="panda" rpy="0 ${0} ${pi}" xyz="0 0.00 -0.000" connected_to="panda_link8"/>
 </robot>

File: data/xacro/push.xacro (robot description, xacro)
@@ -11,5 +11,5 @@
         <parent link="${ns}_push"/>
         <child link="${ns}_push_ref"/>
-        <origin rpy="0.0 0.0 0.0" xyz="0 0 0.188"/>
+        <origin rpy="0.0 0.0 0.0" xyz="0 0 0.18"/>
       </joint>
     </xacro:unless>
@@ -25,5 +25,5 @@
       </inertial>
       <visual>
-        <origin xyz="${xyz}" rpy="0 0 0"/>
+        <origin xyz="${xyz}" rpy="${rpy}"/>
         <geometry>
           <mesh filename="file://@MESHES_DESTINATION@/push.stl" />
@@ -34,5 +34,5 @@
       </visual>
       <collision>
-        <origin xyz="${xyz}" rpy="0 0 0"/>
+        <origin xyz="${xyz}" rpy="${rpy}"/>
         <geometry>
           <mesh filename="file://@MESHES_DESTINATION@/push.stl" />
