Commit message: Minor PandaPush-change Tool Version

File: data/xacro/push.xacro (robot description, xacro)
@@ -11,5 +11,5 @@
         <parent link="${ns}_push"/>
         <child link="${ns}_push_ref"/>
-        <origin rpy="0.0 0.0 0.0" xyz="0 0 0.2"/>
+        <origin rpy="0.0 0.0 0.0" xyz="0 0 0.188"/>
       </joint>
     </xacro:unless>

Commit message: minor: collision on tip of poke tool

File: data/xacro/push.xacro (robot description, xacro)
@@ -41,4 +41,10 @@
     </link>
     <link name="${ns}_push_ref">
+      <collision>
+        <origin xyz="-0.00 0 0.00" rpy="0 0 0"/>
+        <geometry>
+          <sphere radius="${0.012}" />
+        </geometry>
+      </collision>
   </link>
   </xacro:macro>

Commit message: minor push robot

File: data/xacro/push.xacro (robot description, xacro)
@@ -44,5 +44,5 @@
         <origin xyz="-0.00 0 0.00" rpy="0 0 0"/>
         <geometry>
-          <sphere radius="${0.012}" />
+          <sphere radius="${0.02}" />
         </geometry>
       </collision>
