Commit message: minor

File: data/xacro/pump.xacro (robot description, xacro)
@@ -11,5 +11,5 @@
         <parent link="${ns}_pump"/>
         <child link="${ns}_pump_ref"/>
-        <origin rpy="0 0 -0.7853981633974483" xyz="0 0 0.11"/>
+        <origin rpy="0 0 0.0" xyz="0 0 0.145"/>
       </joint>
     </xacro:unless>

Commit message: minor-adapt succion cup frame  to the nondeformable Part

File: data/xacro/pump.xacro (robot description, xacro)
@@ -11,5 +11,6 @@
         <parent link="${ns}_pump"/>
         <child link="${ns}_pump_ref"/>
-        <origin rpy="0 0 0.0" xyz="0 0 0.145"/>
+        <!-- <origin rpy="0 0 0.0" xyz="0 0 0.145"/> -->
+        <origin rpy="0 0 0.0" xyz="0 0 0.11"/>
       </joint>
     </xacro:unless>

Commit message: minor adding suction cup to define frames

File: data/xacro/pump.xacro (robot description, xacro)
@@ -13,4 +13,16 @@
         <!-- <origin rpy="0 0 0.0" xyz="0 0 0.145"/> -->
         <origin rpy="0 0 0.0" xyz="0 0 0.11"/>
+      </joint>
+      <joint name="${ns}_fixsuction_joint_ref" type="fixed">
+        <parent link="${ns}_pump"/>
+        <child link="${ns}_fixsuction_ref"/>
+        <!-- <origin rpy="0 0 0.0" xyz="0 0 0.145"/> -->
+        <origin rpy="0 0 0.0" xyz="0 0 0.10"/>
+      </joint>
+      <joint name="${ns}_NDsuction_joint_ref" type="fixed">
+        <parent link="${ns}_fixsuction_ref"/>
+        <child link="${ns}_NDsuction_ref"/>
+        <!-- <origin rpy="0 0 0.0" xyz="0 0 0.145"/> -->
+        <origin rpy="0 0 0.0" xyz="0 0 -0.009"/>
       </joint>
     </xacro:unless>
@@ -43,23 +55,36 @@
     </link>
     <link name="${ns}_pump_ref">
-        <!--collision>
-          <origin rpy="3.141592653589793 1.5707963267948966 1.5707963267948966" xyz="0.0424 0.0424 0.0"/>
-          <geometry>
-            <cylinder length="0.01" radius="0.06"/>
-          </geometry>
-        </collision>
-            <collision>
-      <origin rpy="0 0 0" xyz="0.0424 0.0424 -0.02"/>
-      <geometry>
-        <sphere radius="0.06"/>
-      </geometry>
-    </collision>
-    <collision>
-      <origin rpy="0 0 0" xyz="0.0424 0.0424 -0.03"/>
-      <geometry>
-        <sphere radius="0.06"/>
-      </geometry>
-    </collision-->
-    <!--  scale="0.001 0.001 0.001" -->
+    </link>
+    <link name="${ns}_fixsuction_ref">
+      <inertial>
+        <mass value="0.013" />
+        <origin xyz="0 0 0.00" rpy="0 0 0" />
+        <inertia ixx="0.001" ixy="0.0" ixz="0.0" iyy="0.001" iyz="0.0" izz="0.001" />
+      </inertial>
+      <visual>
+        <origin xyz="${xyz}" rpy="3.14 0 0"/>
+        <geometry>
+          <mesh filename="file:@MESHES_DESTINATION@/sc_fixation.stl" />
+        </geometry>
+        <material name="">
+          <color rgba="0.2 0.2 0.2 1.0"/>
+        </material>
+      </visual>
+    </link>
+    <link name="${ns}_NDsuction_ref">
+      <inertial>
+        <mass value="0.0105" />
+        <origin xyz="0 0 0.00" rpy="0 0 0" />
+        <inertia ixx="0.001" ixy="0.0" ixz="0.0" iyy="0.001" iyz="0.0" izz="0.001" />
+      </inertial>
+      <visual>
+        <origin xyz="${xyz}" rpy="3.14 0 0"/>
+        <geometry>
+          <mesh filename="file:@MESHES_DESTINATION@/suction_cup.stl" />
+        </geometry>
+        <material name="">
+          <color rgba="0.0 1.0 0.0 1.0"/>
+        </material>
+      </visual>
     </link>
   </xacro:macro>

Commit message: minor: place frame on contact surface

File: data/xacro/pump.xacro (robot description, xacro)
@@ -12,5 +12,5 @@
         <child link="${ns}_pump_ref"/>
         <!-- <origin rpy="0 0 0.0" xyz="0 0 0.145"/> -->
-        <origin rpy="0 0 0.0" xyz="0 0 0.11"/>
+        <origin rpy="0 0 0.0" xyz="0 0 0.14"/>
       </joint>
       <joint name="${ns}_fixsuction_joint_ref" type="fixed">

Commit message: minor adding suction cup details

File: data/xacro/pump.xacro (robot description, xacro)
@@ -8,15 +8,15 @@
         <origin xyz="${xyz}" rpy="${rpy}"/>
       </joint>
-      <joint name="${ns}_pump_joint_ref" type="fixed">
+      <joint name="${ns}_flanpump_joint_ref" type="fixed">
         <parent link="${ns}_pump"/>
-        <child link="${ns}_pump_ref"/>
+        <child link="${ns}_flanpump"/>
         <!-- <origin rpy="0 0 0.0" xyz="0 0 0.145"/> -->
-        <origin rpy="0 0 0.0" xyz="0 0 0.14"/>
+        <origin rpy="0 0 0.0" xyz="0 0 0.09"/>
       </joint>
       <joint name="${ns}_fixsuction_joint_ref" type="fixed">
-        <parent link="${ns}_pump"/>
+        <parent link="${ns}_flanpump"/>
         <child link="${ns}_fixsuction_ref"/>
         <!-- <origin rpy="0 0 0.0" xyz="0 0 0.145"/> -->
-        <origin rpy="0 0 0.0" xyz="0 0 0.10"/>
+        <origin rpy="0 0 0.0" xyz="0 0 0.03"/>
       </joint>
       <joint name="${ns}_NDsuction_joint_ref" type="fixed">
@@ -25,4 +25,10 @@
         <!-- <origin rpy="0 0 0.0" xyz="0 0 0.145"/> -->
         <origin rpy="0 0 0.0" xyz="0 0 -0.009"/>
+      </joint>
+      <joint name="${ns}_pump_joint_ref" type="fixed">
+        <parent link="${ns}_flanpump"/>
+        <child link="${ns}_pump_ref"/>
+        <!-- <origin rpy="0 0 0.0" xyz="0 0 0.145"/> -->
+        <origin rpy="0 0 0.0" xyz="0 0 0.072"/>
       </joint>
     </xacro:unless>
@@ -55,4 +61,20 @@
     </link>
     <link name="${ns}_pump_ref">
+    </link>
+    <link name="${ns}_flanpump">
+      <inertial>
+        <mass value="0.05" />
+        <origin xyz="0 0 0.00" rpy="0 0 0" />
+        <inertia ixx="0.001" ixy="0.0" ixz="0.0" iyy="0.001" iyz="0.0" izz="0.001" />
+      </inertial>
+      <visual>
+        <origin xyz="${xyz}" rpy="3.14 0 0"/>
+        <geometry>
+          <mesh filename="file:@MESHES_DESTINATION@/flanpump.stl" />
+        </geometry>
+        <material name="">
+          <color rgba="0.2 0.2 0.2 1.0"/>
+        </material>
+      </visual>
     </link>
     <link name="${ns}_fixsuction_ref">
